File: PCB/KICAD_PROJECT/Hackpad.kicad_pcb (KiCad board)
At the start: 2 copper layers, 62 x 89 mm, 21 parts, among them J1 OLED_128x64, SW1 RotaryEncoder_Switch, U1 MCU_Seeed_XIAO_RP2040

Commit message: Fixed routing flaw
Connections:
- SW1 pad C: GROUND -> 3.3V
- U1 pad 12: unconnected-(U1-3V3-Pad12) -> 3.3V
Routing:
- net 3.3V: track 0.00 -> 106.9 mm
- net GROUND: track 150.3 -> 134.7 mm
