File: PCB/KICAD_PROJECT/Hackpad.kicad_sch (KiCad schematic)
At the start: 21 parts, among them J1 OLED_128x64, SW1 RotaryEncoder_Switch, U1 MCU_Seeed_XIAO_RP2040

Commit message: Fixed routing flaw
Parts:
- added D10: Diode, ScottoKeebs_Components:Diode_DO-35, symbol ScottoKeebs:Placeholder_Diode
- added S10: Keyswitch, ScottoKeebs_Hotswap:Hotswap_MX_1.00u, symbol ScottoKeebs:Placeholder_Keyswitch
Connections:
- net RTRY A is gone; now on net ROW 2: SW1.A, U1.11 (PA6_A10_D10_MOSI)
- net RTRY B is gone; now on net ROW 2: SW1.B, U1.10 (PA5_A9_D9_MISO)
- net RTRY SWITCH is gone; now on net ROW 2: SW1.S2, U1.9 (PA7_A8_D8_SCK)
- net GROUND: now also S10.1
- net ROW 2: now also U1.12 (3V3), D10.1 (K)
- new net: D10.2 (A), S10.2
